Commit message: Add files via upload

File: src/thorvald_2d_nav/urdf/model.urdf (robot description, URDF)
Before this commit: robot thorvald_ii, 18 links, 17 joints
Joints:
- joint hokuyo_joint: origin xyz=0.42 0 0.2 rpy=0 0 0 -> xyz=0.02 0 0.2 rpy=0 0 0; parent base_link -> front_link

File: src/thorvald_2d_nav/urdf/trolley.urdf (robot description, URDF)
Before this commit: robot trolley, 8 links, 7 joints
Links:
- removed link RTK_left_antenna
- removed link RTK_right_antenna
- removed link xsens_imu
- added link base_imu_link; visual box size=0.05 0.05 0.02
- added link gps; visual box size=0.05 0.05 0.02
- added link laser, mass 1e-5; collision box size=0.1 0.1 0.1; visual mesh filename=package://testbot_description/meshes/hokuyo.dae
Joints:
- removed joint center_to_xsens_imu
- removed joint down_right_corner_to_RTK_right_antenna
- removed joint top_left_corner_to_RTK_left_antenna
- added joint center_to_gps: type fixed, parent base_link, child gps, origin xyz=0.28 0.0 0.01
- added joint center_to_imu: type fixed, parent base_link, child base_imu_link, origin xyz=-0.28 0.0 0.01
- added joint hokuyo_joint: type fixed, parent base_link, child laser, origin xyz=0.02 0 0.2 rpy=0 0 0, axis 0 1 0
